Commit message: removed unnecessary macro parameters

File: xacro/hokuyo.urdf.xacro (robot description, xacro)
@@ -1,6 +1,5 @@
 <?xml version="1.0"?>
 <robot name="sensor_hokuyo_ust10lx" xmlns:xacro="http://wiki.ros.org/xacro">
-	<xacro:macro name="sensor_hokuyo_ust10lx"
-		params="prefix parent prefix_topic:='front_laser' *origin min_angle:=-2.3562 max_angle:=2.3562 gpu:=^|true">
+	<xacro:macro name="sensor_hokuyo_ust10lx" params="prefix parent *origin ">
 		<joint name="${prefix}_base_joint" type="fixed">
 			<xacro:insert_block name="origin" />
@@ -35,5 +34,6 @@
 		</link>
 	</xacro:macro>
-<!--
+	<!-- default values:  topic = front_laser | rear_laser min_angle:=-2.3562 max_angle:=2.3562 gpu:=^|true -->
+	<!--
 	<xacro:macro name="sensor_hokuyo_ust10_gazebo">
 		<gazebo reference="${prefix}_link">
@@ -80,4 +80,5 @@
 			</sensor>
 		</gazebo>
-	</xacro:macro>-->
+	</xacro:macro>
+	-->
 </robot>

File: xacro/zed.urdf.xacro (robot description, xacro)
@@ -82,5 +82,6 @@
 		<link name="${prefix}_right_camera_optical_frame" />
 	</xacro:macro>
-	<!-- default values: format:=R8G8B8 near:=0.05 far:=2500
+	<!-- default values: format:=R8G8B8 near:=0.05 far:=2500 -->
+	<!--
 	<xacro:macro name="sensor_zed" params="prefix:=myzed parent *origin model:=zed">
 		<xacro:sensor_zed prefix="${prefix}" parent="${parent}" model="${model}">
@@ -157,13 +158,15 @@
 	</xacro:macro>
 	-->
-	<!--<xacro:stereo_camera
-			prefix="${prefix}"
-			hfov="1.2217"
-			baseline="${baseline}"
-			fps="40"
-			width="640"
-			height="480"
-			format="${format}"
-			near="${near}"
-			far="${far}" />-->
+	<!--
+	<xacro:stereo_camera
+		prefix="${prefix}"
+		hfov="1.2217"
+		baseline="${baseline}"
+		fps="40"
+		width="640"
+		height="480"
+		format="${format}"
+		near="${near}"
+		far="${far}" />
+	-->
 </robot>
