Commit message: Added lidar plugin

File: xacro/VLP-16.urdf.xacro (robot description, xacro)
@@ -52,5 +52,5 @@
       <collision>
         <geometry>
-          <sphere radius="0"/>
+          <sphere radius="0.00001"/>
         </geometry>
       </collision>
@@ -149,4 +149,37 @@
       </xacro:unless>
     </gazebo>
+  <!-- <gazebo reference="${name}">
+    <sensor name="lidar" type='gpu_lidar'>
+            <pose>0 0 1.0 0 0 0</pose>
+            <topic>scan</topic>
+            <update_rate>10</update_rate>
+            <ray>
+                <scan>
+                    <horizontal>
+                        <samples>5</samples>
+                        <min_angle>-0.349066</min_angle>
+                        <max_angle>0.349066</max_angle>
+                    </horizontal>
+                    <vertical>
+                        <samples>5</samples>
+                        <min_angle>-0.174533</min_angle>
+                        <max_angle>0.174533</max_angle>
+                    </vertical>
+                </scan>
+                <range>
+                    <min>0.1</min>
+                    <max>2.0</max>
+                    <resolution>0.01</resolution>
+                </range>
+            </ray>
+            <always_on>1</always_on>
+            <visualize>true</visualize>
+          <plugin
+            filename="libignition-gazebo-sensors-system.so"
+            name="ignition::gazebo::systems::Sensors">
+            <render_engine>ogre2</render_engine>
+          </plugin>
+        </sensor>
+    </gazebo> -->
   </xacro:macro>
 </robot>

Commit message: Added ignition fortrees plugin

File: xacro/VLP-16.urdf.xacro (robot description, xacro)
@@ -3,4 +3,6 @@
   <xacro:property name="M_PI" value="3.1415926535897931" />
   <xacro:macro name="VLP-16" params="*origin parent:=base_link name:=velodyne tf_prefix:='' topic:=/velodyne_points organize_cloud:=false hz:=10 lasers:=16 samples:=1875 collision_range:=0.3 min_range:=0.9 max_range:=130.0 noise:=0.008 min_angle:=-${M_PI} max_angle:=${M_PI} gpu:=false">
+  <xacro:arg name="ign" default="false"/>
+  <xacro:property name="ign" value="$(arg ign)"/>
     <joint name="${name}_base_mount_joint" type="fixed">
       <xacro:insert_block name="origin" />
@@ -57,11 +59,13 @@
     </link>
     <!-- Gazebo requires the velodyne_gazebo_plugins package -->
-    <gazebo reference="${name}">
-      <xacro:if value="${gpu}">
-        <sensor type="gpu_ray" name="${name}-VLP16">
-          <pose>0 0 0 0 0 0</pose>
-          <visualize>false</visualize>
+    <xacro:if value="${ign}">
+      <gazebo reference="${name}">
+        <sensor name="${name}-VLP16" type="gpu_lidar">
           <update_rate>${hz}</update_rate>
-          <ray>
+          <visualize>true</visualize>
+          <always_on>true</always_on>
+          <ignition_frame_id>${name}</ignition_frame_id>
+          <topic>${topic}</topic>
+          <lidar>
             <scan>
               <horizontal>
@@ -88,97 +92,136 @@
               <stddev>0.0</stddev>
             </noise>
-          </ray>
-          <plugin name="gazebo_ros_laser_controller" filename="libgazebo_ros_velodyne_laser.so">
-            <ros>
-              <namespace>/${name}</namespace>
-              <remapping>~/out:=${topic}</remapping>
-            </ros>
-            <tf_prefix>${tf_prefix}</tf_prefix>
-            <frame_name>${name}</frame_name>
-            <organize_cloud>${organize_cloud}</organize_cloud>
-            <min_range>${min_range}</min_range>
-            <max_range>${max_range}</max_range>
-            <gaussian_noise>${noise}</gaussian_noise>
-          </plugin>
+          </lidar>
         </sensor>
-      </xacro:if>
-      <xacro:unless value="${gpu}">
-        <sensor type="ray" name="${name}-VLP16">
-          <pose>0 0 0 0 0 0</pose>
-          <visualize>false</visualize>
-          <update_rate>${hz}</update_rate>
-          <ray>
-            <scan>
-              <horizontal>
-                <samples>${samples}</samples>
-                <resolution>1</resolution>
-                <min_angle>${min_angle}</min_angle>
-                <max_angle>${max_angle}</max_angle>
-              </horizontal>
-              <vertical>
-                <samples>${lasers}</samples>
-                <resolution>1</resolution>
-                <min_angle>-${15.0*M_PI/180.0}</min_angle>
-                <max_angle> ${15.0*M_PI/180.0}</max_angle>
-              </vertical>
-            </scan>
-            <range>
-              <min>${collision_range}</min>
-              <max>${max_range+1}</max>
-              <resolution>0.001</resolution>
-            </range>
-            <noise>
-              <type>gaussian</type>
-              <mean>0.0</mean>
-              <stddev>0.0</stddev>
-            </noise>
-          </ray>
-          <plugin name="gazebo_ros_laser_controller" filename="libgazebo_ros_velodyne_laser.so">
-            <ros>
-              <namespace>/${name}</namespace>
-              <remapping>~/out:=${topic}</remapping>
-            </ros>
-            <tf_prefix>${tf_prefix}</tf_prefix>
-            <frame_name>${name}</frame_name>
-            <organize_cloud>${organize_cloud}</organize_cloud>
-            <min_range>${min_range}</min_range>
-            <max_range>${max_range}</max_range>
-            <gaussian_noise>${noise}</gaussian_noise>
-          </plugin>
-        </sensor>
-      </xacro:unless>
-    </gazebo>
-  <!-- <gazebo reference="${name}">
-    <sensor name="lidar" type='gpu_lidar'>
-            <pose>0 0 1.0 0 0 0</pose>
-            <topic>scan</topic>
-            <update_rate>10</update_rate>
+      </gazebo>
+    </xacro:if>
+    <xacro:unless value="${ign}">
+      <gazebo reference="${name}">
+        <xacro:if value="${gpu}">
+          <sensor type="gpu_ray" name="${name}-VLP16">
+            <pose>0 0 0 0 0 0</pose>
+            <visualize>false</visualize>
+            <update_rate>${hz}</update_rate>
             <ray>
-                <scan>
-                    <horizontal>
-                        <samples>5</samples>
-                        <min_angle>-0.349066</min_angle>
-                        <max_angle>0.349066</max_angle>
-                    </horizontal>
-                    <vertical>
-                        <samples>5</samples>
-                        <min_angle>-0.174533</min_angle>
-                        <max_angle>0.174533</max_angle>
-                    </vertical>
-                </scan>
-                <range>
-                    <min>0.1</min>
-                    <max>2.0</max>
-                    <resolution>0.01</resolution>
-                </range>
+              <scan>
+                <horizontal>
+                  <samples>${samples}</samples>
+                  <resolution>1</resolution>
+                  <min_angle>${min_angle}</min_angle>
+                  <max_angle>${max_angle}</max_angle>
+                </horizontal>
+                <vertical>
+                  <samples>${lasers}</samples>
+                  <resolution>1</resolution>
+                  <min_angle>-${15.0*M_PI/180.0}</min_angle>
+                  <max_angle> ${15.0*M_PI/180.0}</max_angle>
+                </vertical>
+              </scan>
+              <range>
+                <min>${collision_range}</min>
+                <max>${max_range+1}</max>
+                <resolution>0.001</resolution>
+              </range>
+              <noise>
+                <type>gaussian</type>
+                <mean>0.0</mean>
+                <stddev>0.0</stddev>
+              </noise>
             </ray>
-            <always_on>1</always_on>
-            <visualize>true</visualize>
-          <plugin
-            filename="libignition-gazebo-sensors-system.so"
-            name="ignition::gazebo::systems::Sensors">
-            <render_engine>ogre2</render_engine>
-          </plugin>
-        </sensor>
+            <plugin name="gazebo_ros_laser_controller" filename="libgazebo_ros_velodyne_laser.so">
+              <ros>
+                <namespace>/${name}</namespace>
+                <remapping>~/out:=${topic}</remapping>
+              </ros>
+              <tf_prefix>${tf_prefix}</tf_prefix>
+              <frame_name>${name}</frame_name>
+              <organize_cloud>${organize_cloud}</organize_cloud>
+              <min_range>${min_range}</min_range>
+              <max_range>${max_range}</max_range>
+              <gaussian_noise>${noise}</gaussian_noise>
+            </plugin>
+          </sensor>
+        </xacro:if>
+        <xacro:unless value="${gpu}">
+          <sensor type="ray" name="${name}-VLP16">
+            <pose>0 0 0 0 0 0</pose>
+            <visualize>false</visualize>
+            <update_rate>${hz}</update_rate>
+            <ray>
+              <scan>
+                <horizontal>
+                  <samples>${samples}</samples>
+                  <resolution>1</resolution>
+                  <min_angle>${min_angle}</min_angle>
+                  <max_angle>${max_angle}</max_angle>
+                </horizontal>
+                <vertical>
+                  <samples>${lasers}</samples>
+                  <resolution>1</resolution>
+                  <min_angle>-${15.0*M_PI/180.0}</min_angle>
+                  <max_angle> ${15.0*M_PI/180.0}</max_angle>
+                </vertical>
+              </scan>
+              <range>
+                <min>${collision_range}</min>
+                <max>${max_range+1}</max>
+                <resolution>0.001</resolution>
+              </range>
+              <noise>
+                <type>gaussian</type>
+                <mean>0.0</mean>
+                <stddev>0.0</stddev>
+              </noise>
+            </ray>
+            <plugin name="gazebo_ros_laser_controller" filename="libgazebo_ros_velodyne_laser.so">
+              <ros>
+                <namespace>/${name}</namespace>
+                <remapping>~/out:=${topic}</remapping>
+              </ros>
+              <tf_prefix>${tf_prefix}</tf_prefix>
+              <frame_name>${name}</frame_name>
+              <organize_cloud>${organize_cloud}</organize_cloud>
+              <min_range>${min_range}</min_range>
+              <max_range>${max_range}</max_range>
+              <gaussian_noise>${noise}</gaussian_noise>
+            </plugin>
+          </sensor>
+        </xacro:unless>
+      </gazebo>
+    </xacro:unless>
+    <!-- <gazebo reference="${name}">
+      <sensor name="${name}-VLP16" type="gpu_lidar">
+        <update_rate>${hz}</update_rate>
+        <visualize>true</visualize>
+        <always_on>true</always_on>
+        <ignition_frame_id>${name}</ignition_frame_id>
+        <topic>${topic}</topic>
+        <lidar>
+          <scan>
+            <horizontal>
+              <samples>${samples}</samples>
+              <resolution>1</resolution>
+              <min_angle>${min_angle}</min_angle>
+              <max_angle>${max_angle}</max_angle>
+            </horizontal>
+            <vertical>
+              <samples>${lasers}</samples>
+              <resolution>1</resolution>
+              <min_angle>-${15.0*M_PI/180.0}</min_angle>
+              <max_angle> ${15.0*M_PI/180.0}</max_angle>
+            </vertical>
+          </scan>
+          <range>
+            <min>${collision_range}</min>
+            <max>${max_range+1}</max>
+            <resolution>0.001</resolution>
+          </range>
+          <noise>
+            <type>gaussian</type>
+            <mean>0.0</mean>
+            <stddev>0.0</stddev>
+          </noise>
+        </lidar>
+      </sensor>
     </gazebo> -->
   </xacro:macro>
