Commit message: Code comments deleted

File: xacro/VLP-16.urdf.xacro (robot description, xacro)
@@ -58,5 +58,4 @@
       </collision>
     </link>
-    <!-- Gazebo requires the velodyne_gazebo_plugins package -->
     <xacro:if value="${ign}">
       <gazebo reference="${name}">

File: xacro/hokuyo.urdf.xacro (robot description, xacro)
@@ -34,51 +34,3 @@
 		</link>
 	</xacro:macro>
-	<!-- default values:  topic = front_laser | rear_laser min_angle:=-2.3562 max_angle:=2.3562 gpu:=^|true -->
-	<!--
-	<xacro:macro name="sensor_hokuyo_ust10_gazebo">
-		<gazebo reference="${prefix}_link">
-			<xacro:if value="${gpu}">
-				<xacro:property name="ray_type" value="gpu_ray" />
-				<xacro:property name="plugin_lib" value="libgazebo_ros_gpu_laser.so" />
-			</xacro:if>
-			<xacro:unless value="${gpu}">
-				<xacro:property name="ray_type" value="ray" />
-				<xacro:property name="plugin_lib" value="libgazebo_ros_ray_laser.so" />
-			</xacro:unless>
-			<sensor type="${ray_type}" name="${prefix}_sensor">
-				<pose>0 0 0 0 0 0</pose>
-				<visualize>false</visualize>
-				<update_rate>40</update_rate>
-				<ray>
-					<scan>
-						<horizontal>
-							<samples>1081</samples>
-							<resolution>1</resolution>
-							<min_angle>${min_angle}</min_angle>
-							<max_angle>${max_angle}</max_angle>
-						</horizontal>
-					</scan>
-					<range>
-						<min>0.06</min>
-						<max>10.0</max>
-						<resolution>0.004359297</resolution>
-					</range>
-					<noise>
-						<type>gaussian</type>
-						<mean>0.0</mean>
-						<stddev>0.01</stddev>
-					</noise>
-				</ray>
-				<plugin name="${prefix}_controller" filename="libgazebo_ros_ray_sensor.so">
-					<ros>
-						<remapping>~/out:=${prefix_topic}/scan</remapping>
-					</ros>
-					when leaving away frame_name it defaults to base_footprint instead
-					<frame_name>${prefix}_link</frame_name>
-					<output_type>sensor_msgs/LaserScan</output_type>
-				</plugin>
-			</sensor>
-		</gazebo>
-	</xacro:macro>
-	-->
 </robot>

File: xacro/imu.urdf.xacro (robot description, xacro)
@@ -1,7 +1,4 @@
 <?xml version="1.0"?>
 <robot name="sensor_imu" xmlns:xacro="http://wiki.ros.org/xacro">
-	<!-- Solid cuboid of width w, height h, depth d, and mass m -->
-	<!-- w relates to X axis, d to Z axis, and h to Y axis -->
-	<!-- Keep this comment -->
 	<xacro:macro name="solid_cuboid_inertia" params="m w h d">
 		<inertia ixx="${(m*(h*h+d*d))/12}" ixy="0" ixz="0"

File: xacro/orbbec_astra.urdf.xacro (robot description, xacro)
@@ -51,35 +51,3 @@
 		<link name="${prefix}_depth_optical_frame" />
 	</xacro:macro>
-	<!--
-	<xacro:macro name="sensor_orbbec_astra_gazebo" params="ns prefix">
-		<xacro:property name="deg_to_rad" value="0.01745329251994329577" />
-		<gazebo reference="${prefix}_link">
-			<sensor name="${prefix}" type="depth">
-				<pose>0 0 0 0 0 0</pose>
-				<visualize>false</visualize>
-				<update_rate>30</update_rate>
-				<camera>
-					<horizontal_fov>1,04719755</horizontal_fov>
-					<vertical_fov>0.86393798</vertical_fov>
-					<image>
-						<format>B8G8R8</format>
-						<width>640</width>
-						<height>480</height>
-					</image>
-					<clip>
-						<near>0.05</near>
-						<far>100.0</far>
-					</clip>
-				</camera>
-				<plugin name="${prefix}" filename="libgazebo_ros_camera.so">
-					<ros>
-						<namespace>${ns}</namespace>
-					</ros>
-					<frame_name>${ns}/${prefix}_rgb_optical_frame</frame_name>
-					<min_depth>0.4</min_depth>
-					<max_depth>6.5</max_depth>
-				</plugin>
-			</sensor>
-		</gazebo>
-	</xacro:macro>-->
 </robot>

File: xacro/realsense_d430.gazebo.xacro (robot description, xacro)
@@ -1,7 +1,5 @@
 <?xml version="1.0"?>
-<!-- Copyright (C) 2024, Federico Rollo -->
 <robot xmlns:xacro="http://ros.org/wiki/xacro">
   <xacro:macro name="gazebo_d430" params="camera_name reference_link topics_ns depth_optical_frame color_optical_frame infrared1_optical_frame infrared2_optical_frame" >
-    <!-- Load parameters to model's main link-->
     <xacro:property name="deg_to_rad" value="0.01745329251994329577" />
     <gazebo reference="${reference_link}">
@@ -9,14 +7,8 @@
       <enable_wind>0</enable_wind>
       <kinematic>0</kinematic>
-<!--      <gravity>1</gravity>-->
-      <!--<mu>1</mu>-->
       <mu2>1</mu2>
       <fdir1>0 0 0</fdir1>
-      <!--<slip1>0</slip1>
-      <slip2>0</slip2>-->
       <kp>1e+13</kp>
       <kd>1</kd>
-      <!--<max_vel>0.01</max_vel>
-      <min_depth>0</min_depth>-->
       <sensor name="${camera_name}color" type="camera">
         <camera name="${camera_name}">

File: xacro/realsense_d430.urdf.xacro (robot description, xacro)
@@ -1,23 +1,14 @@
 <?xml version="1.0"?>
-<!-- Copyright (C) 2024, Federico Rollo -->
 <robot name="realsense_d430" xmlns:xacro="http://ros.org/wiki/xacro">
-  <!--File includes-->
   <xacro:include filename="$(find sensors_description)/xacro/realsense_d430.gazebo.xacro"/>
   <xacro:macro name="realsense_d430" params="name:=camera topics_ns:=camera parent *origin">
     <xacro:property name="M_PI" value="3.1415926535897931" />
-    <!-- The following values are approximate, and the camera node
-     publishing TF values with actual calibrated camera extrinsic values -->
     <xacro:property name="d430_cam_depth_to_left_ir_offset" value="0.0"/>
     <xacro:property name="d430_cam_depth_to_right_ir_offset" value="-0.050"/>
     <xacro:property name="d430_cam_depth_to_color_offset" value="0.015"/>
-    <!-- The following values model the aluminum peripherial case for the
-  	D430 camera, with the camera joint represented by the actual
-  	peripherial camera tripod mount -->
     <xacro:property name="d430_cam_width" value="0.090"/>
     <xacro:property name="d430_cam_height" value="0.025"/>
     <xacro:property name="d430_cam_depth" value="0.02505"/>
     <xacro:property name="d430_cam_mount_from_center_offset" value="0.0149"/>
-    <!-- The following offset is relative the the physical D430 camera peripherial
-  	camera tripod mount -->
     <xacro:property name="d430_cam_depth_px" value="${d430_cam_mount_from_center_offset}"/>
     <xacro:property name="d430_cam_depth_py" value="0.0175"/>
@@ -26,5 +17,4 @@
 	  <color rgba="0.5 0.5 0.5 1"/>
     </material>
-    <!-- camera body, with origin at bottom screw mount -->
     <joint name="${name}_joint" type="fixed">
       <xacro:insert_block name="origin" />
@@ -58,5 +48,4 @@
       </inertial>
     </link>
-    <!-- camera depth joints and links -->
     <joint name="${name}_depth_joint" type="fixed">
       <origin xyz="0 0 0" rpy="0 0 0"/>
@@ -71,5 +60,4 @@
     </joint>
     <link name="${name}_depth_optical_frame"/>
-    <!-- camera left IR joints and links -->
     <joint name="${name}_left_ir_joint" type="fixed">
       <origin xyz="0 ${d430_cam_depth_to_left_ir_offset} 0" rpy="0 0 0" />
@@ -84,5 +72,4 @@
     </joint>
     <link name="${name}_left_ir_optical_frame"/>
-    <!-- camera right IR joints and links -->
     <joint name="${name}_right_ir_joint" type="fixed">
       <origin xyz="0 ${d430_cam_depth_to_right_ir_offset} 0" rpy="0 0 0" />
@@ -97,5 +84,4 @@
     </joint>
     <link name="${name}_right_ir_optical_frame"/>
-    <!-- camera color joints and links -->
     <joint name="${name}_color_joint" type="fixed">
       <origin xyz="0 ${d430_cam_depth_to_color_offset} 0" rpy="0 0 0" />
@@ -110,5 +96,4 @@
     </joint>
     <link name="${name}_color_optical_frame"/>
-    <!-- Realsense Gazebo Plugin -->
     <xacro:gazebo_d430 camera_name="${name}" reference_link="${name}_link" topics_ns="${topics_ns}" depth_optical_frame="${name}_depth_optical_frame" color_optical_frame="${name}_color_optical_frame" infrared1_optical_frame="${name}_left_ir_optical_frame" infrared2_optical_frame="${name}_right_ir_optical_frame"/>
   </xacro:macro>

File: xacro/realsense_d435.gazebo.xacro (robot description, xacro)
@@ -1,7 +1,5 @@
 <?xml version="1.0"?>
-<!-- Copyright (C) 2024, Federico Rollo -->
 <robot xmlns:xacro="http://ros.org/wiki/xacro">
   <xacro:macro name="gazebo_d435" params="camera_name reference_link topics_ns depth_optical_frame color_optical_frame infrared1_optical_frame infrared2_optical_frame" >
-    <!-- Load parameters to model's main link-->
     <xacro:property name="deg_to_rad" value="0.01745329251994329577" />
     <gazebo reference="${reference_link}">
@@ -9,14 +7,8 @@
       <enable_wind>0</enable_wind>
       <kinematic>0</kinematic>
-<!--      <gravity>1</gravity>-->
-      <!--<mu>1</mu>-->
       <mu2>1</mu2>
       <fdir1>0 0 0</fdir1>
-      <!--<slip1>0</slip1>
-      <slip2>0</slip2>-->
       <kp>1e+13</kp>
       <kd>1</kd>
-      <!--<max_vel>0.01</max_vel>
-      <min_depth>0</min_depth>-->
       <sensor name="${camera_name}color" type="camera">
         <camera name="${camera_name}">

File: xacro/realsense_d435.urdf.xacro (robot description, xacro)
@@ -1,23 +1,14 @@
 <?xml version="1.0"?>
-<!-- Copyright (C) 2024, Federico Rollo -->
 <robot name="realsense_d435" xmlns:xacro="http://ros.org/wiki/xacro">
-  <!--File includes-->
   <xacro:include filename="$(find sensors_description)/xacro/realsense_d435.gazebo.xacro"/>
   <xacro:macro name="realsense_d435" params="name:=camera topics_ns:=camera parent *origin">
     <xacro:property name="M_PI" value="3.1415926535897931" />
-    <!-- The following values are approximate, and the camera node
-     publishing TF values with actual calibrated camera extrinsic values -->
     <xacro:property name="d435_cam_depth_to_left_ir_offset" value="0.0"/>
     <xacro:property name="d435_cam_depth_to_right_ir_offset" value="-0.050"/>
     <xacro:property name="d435_cam_depth_to_color_offset" value="0.015"/>
-    <!-- The following values model the aluminum peripherial case for the
-  	D435 camera, with the camera joint represented by the actual
-  	peripherial camera tripod mount -->
     <xacro:property name="d435_cam_width" value="0.090"/>
     <xacro:property name="d435_cam_height" value="0.025"/>
     <xacro:property name="d435_cam_depth" value="0.02505"/>
     <xacro:property name="d435_cam_mount_from_center_offset" value="0.0149"/>
-    <!-- The following offset is relative the the physical D435 camera peripherial
-  	camera tripod mount -->
     <xacro:property name="d435_cam_depth_px" value="${d435_cam_mount_from_center_offset}"/>
     <xacro:property name="d435_cam_depth_py" value="0.0175"/>
@@ -26,5 +17,4 @@
 	  <color rgba="0.5 0.5 0.5 1"/>
     </material>
-    <!-- camera body, with origin at bottom screw mount -->
     <joint name="${name}_joint" type="fixed">
       <xacro:insert_block name="origin" />
@@ -53,5 +43,4 @@
       </collision>
       <inertial>
-        <!-- The following are not reliable values, and should not be used for modeling -->
         <mass value="0.564" />
         <origin xyz="0 0 0" />
@@ -59,5 +48,4 @@
       </inertial>
     </link>
-    <!-- camera depth joints and links -->
     <joint name="${name}_depth_joint" type="fixed">
       <origin xyz="0 0 0" rpy="0 0 0"/>
@@ -72,5 +60,4 @@
     </joint>
     <link name="${name}_depth_optical_frame"/>
-    <!-- camera left IR joints and links -->
     <joint name="${name}_left_ir_joint" type="fixed">
       <origin xyz="0 ${d435_cam_depth_to_left_ir_offset} 0" rpy="0 0 0" />
@@ -85,5 +72,4 @@
     </joint>
     <link name="${name}_left_ir_optical_frame"/>
-    <!-- camera right IR joints and links -->
     <joint name="${name}_right_ir_joint" type="fixed">
       <origin xyz="0 ${d435_cam_depth_to_right_ir_offset} 0" rpy="0 0 0" />
@@ -98,5 +84,4 @@
     </joint>
     <link name="${name}_right_ir_optical_frame"/>
-    <!-- camera color joints and links -->
     <joint name="${name}_color_joint" type="fixed">
       <origin xyz="0 ${d435_cam_depth_to_color_offset} 0" rpy="0 0 0" />
@@ -111,5 +96,4 @@
     </joint>
     <link name="${name}_color_optical_frame"/>
-    <!-- Realsense Gazebo Plugin -->
     <xacro:gazebo_d435 camera_name="${name}" reference_link="${name}_link" topics_ns="${topics_ns}" depth_optical_frame="${name}_depth_optical_frame" color_optical_frame="${name}_color_optical_frame" infrared1_optical_frame="${name}_left_ir_optical_frame" infrared2_optical_frame="${name}_right_ir_optical_frame"/>
   </xacro:macro>

File: xacro/realsense_d455.gazebo.xacro (robot description, xacro)
@@ -1,8 +1,6 @@
 <?xml version="1.0"?>
-<!-- Copyright (C) 2024, Federico Rollo -->
 <robot xmlns:xacro="http://ros.org/wiki/xacro">
   <xacro:macro name="gazebo_d455" params="camera_name reference_link topics_ns
   depth_optical_frame color_optical_frame infrared1_optical_frame infrared2_optical_frame" >
-    <!-- Load parameters to model's main link-->
     <xacro:property name="deg_to_rad" value="0.01745329251994329577" />
     <gazebo reference="${reference_link}">

File: xacro/realsense_d455.urdf.xacro (robot description, xacro)
@@ -1,29 +1,17 @@
 <?xml version="1.0"?>
-<!-- Copyright (C) 2024, Federico Rollo -->
 <robot name="sensor_d455" xmlns:xacro="http://ros.org/wiki/xacro">
-  <!--File includes-->
   <xacro:include filename="$(find sensors_description)/xacro/realsense_d455.gazebo.xacro"/>
   <xacro:macro name="sensor_d455" params="name:=camera topics_ns:=camera parent *origin">
     <xacro:property name="M_PI" value="3.1415926535897931" />
-    <!-- The following values are approximate, and the camera node
-     publishing TF values with actual calibrated camera extrinsic values -->
     <xacro:property name="d455_cam_depth_to_infra1_offset" value="0.0"/>
     <xacro:property name="d455_cam_depth_to_infra2_offset" value="-0.095"/>
     <xacro:property name="d455_cam_depth_to_color_offset" value="-0.059"/>
-    <!-- The following values model the aluminum peripherial case for the
-  	d455 camera, with the camera joint represented by the actual
-  	peripherial camera tripod mount -->
     <xacro:property name="d455_cam_width" value="0.124"/>
     <xacro:property name="d455_cam_height" value="0.029"/>
     <xacro:property name="d455_cam_depth" value="0.026"/>
     <xacro:property name="d455_cam_mount_from_center_offset" value="0.0158"/>
-    <!-- glass cover is 0.1 mm inwards from front aluminium plate -->
     <xacro:property name="d455_glass_to_front" value="0.1e-3"/>
-    <!-- see datasheet Revision 009, Fig. 4-4 page 68 -->
     <xacro:property name="d455_zero_depth_to_glass" value="4.55e-3"/>
-    <!-- convenience precomputation to avoid clutter-->
     <xacro:property name="d455_mesh_x_offset" value="${d455_cam_mount_from_center_offset-d455_glass_to_front-d455_zero_depth_to_glass}"/>
-    <!-- The following offset is relative to the physical d455 camera peripherial
-  	camera tripod mount -->
     <xacro:property name="d455_cam_depth_px" value="${d455_cam_mount_from_center_offset}"/>
     <xacro:property name="d455_cam_depth_py" value="0.0475"/>
@@ -32,5 +20,4 @@
 	  <color rgba="0.5 0.5 0.5 1"/>
     </material>
-    <!-- camera body, with origin at bottom screw mount -->
     <joint name="${name}_joint" type="fixed">
       <xacro:insert_block name="origin" />
@@ -59,5 +46,4 @@
       </collision>
       <inertial>
-        <!-- The following are not reliable values, and should not be used for modeling -->
         <mass value="0.072" />
         <origin xyz="0 0 0" />
@@ -65,5 +51,4 @@
       </inertial>
     </link>
-    <!-- camera depth joints and links -->
     <joint name="${name}_depth_joint" type="fixed">
       <origin xyz="0 0 0" rpy="0 0 0"/>
@@ -78,5 +63,4 @@
     </joint>
     <link name="${name}_depth_optical_frame"/>
-    <!-- camera left IR joints and links -->
     <joint name="${name}_infra1_joint" type="fixed">
       <origin xyz="0 ${d455_cam_depth_to_infra1_offset} 0" rpy="0 0 0" />
@@ -91,5 +75,4 @@
     </joint>
     <link name="${name}_infra1_optical_frame"/>
-    <!-- camera right IR joints and links -->
     <joint name="${name}_infra2_joint" type="fixed">
       <origin xyz="0 ${d455_cam_depth_to_infra2_offset} 0" rpy="0 0 0" />
@@ -104,5 +87,4 @@
     </joint>
     <link name="${name}_infra2_optical_frame"/>
-    <!-- camera color joints and links -->
     <joint name="${name}_color_joint" type="fixed">
       <origin xyz="0 ${d455_cam_depth_to_color_offset} 0" rpy="0 0 0" />
@@ -117,6 +99,4 @@
     </joint>
     <link name="${name}_color_optical_frame"/>
-    <!-- IMU -->
-    <!-- see datasheet Revision 009, page 114 -->
     <xacro:property name="d455_imu_px" value="-0.01602"/>
     <xacro:property name="d455_imu_py" value="-0.03022"/>
@@ -152,5 +132,4 @@
       <child link="${name}_imu_optical_frame" />
     </joint>
-    <!-- Realsense Gazebo Plugin -->
     <xacro:gazebo_d455 camera_name="${name}" reference_link="${name}_link" topics_ns="${topics_ns}"
       depth_optical_frame="${name}_depth_optical_frame" color_optical_frame="${name}_color_optical_frame"

File: xacro/zed.urdf.xacro (robot description, xacro)
@@ -1,7 +1,4 @@
 <?xml version="1.0"?>
 <robot xmlns:xacro="http://wiki.ros.org/xacro">
-	<!-- Solid cuboid of width w, height h, depth d, and mass m -->
-	<!-- w relates to X axis, d to Z axis, and h to Y axis -->
-	<!-- Keep this comment -->
 	<xacro:macro name="solid_cuboid_inertia" params="m w h d">
 		<inertia ixx="${(m*(h*h+d*d))/12}" ixy="0" ixz="0"
@@ -48,5 +45,4 @@
 			</inertial>
 		</link>
-		<!-- Center camera -->
 		<joint name="${prefix}_camera_center_joint" type="fixed">
 			<parent link="${prefix}_base_link" />
@@ -55,5 +51,4 @@
 		</joint>
 		<link name="${prefix}_camera_center" />
-		<!-- Left camera -->
 		<joint name="${prefix}_camera_left_joint" type="fixed">
 			<origin xyz="0 ${baseline/2} 0" rpy="0 0 0" />
@@ -68,5 +63,4 @@
 		</joint>
 		<link name="${prefix}_left_camera_optical_frame" />
-		<!-- Right camera-->
 		<joint name="${prefix}_camera_right_joint" type="fixed">
 			<origin xyz="0 -${baseline/2} 0" rpy="0 0 0" />
@@ -82,91 +76,3 @@
 		<link name="${prefix}_right_camera_optical_frame" />
 	</xacro:macro>
-	<!-- default values: format:=R8G8B8 near:=0.05 far:=2500 -->
-	<!--
-	<xacro:macro name="sensor_zed" params="prefix:=myzed parent *origin model:=zed">
-		<xacro:sensor_zed prefix="${prefix}" parent="${parent}" model="${model}">
-			<xacro:insert_block name="origin" />
-		</xacro:sensor_zed>
-	</xacro:macro>
-	-->
-	<!--
-	<xacro:macro name="stereo_camera"
-		params="prefix fps baseline hfov width height format near far">
-		<gazebo reference="${prefix}_base_link">
-			<visual>
-				<material>
-					<ambient>0.35 0.35 0.35 1.0</ambient>
-					<diffuse>0.350754 0.350754 0.350754 1.0</diffuse>
-					<specular>0.308273 0.3508273 0.3508273 1.0</specular>
-					<emissive>0.0 0.0 0.0 0.0</emissive>
-				</material>
-			</visual>
-			<sensor type="multicamera" name="stereo_camera">
-				<update_rate>${fps}</update_rate>
-				<camera name="left">
-					<pose>0 0 0 0 0 0 </pose>
-					<horizontal_fov>${hfov}</horizontal_fov>
-					<image>
-						<width>${width}</width>
-						<height>${height}</height>
-						<format>${format}</format>
-					</image>
-					<clip>
-						<near>${near}</near>
-						<far>${far}</far>
-					</clip>
-					<noise>
-						<type>gaussian</type>
-						<mean>0.0</mean>
-						<stddev>0.007</stddev>
-					</noise>
-				</camera>
-				<camera name="right">
-					<pose>${baseline} 0 0 0 0 0</pose>
-					<horizontal_fov>${hfov}</horizontal_fov>
-					<image>
-						<width>${width}</width>
-						<height>${height}</height>
-						<format>${format}</format>
-					</image>
-					<clip>
-						<near>${near}</near>
-						<far>${far}</far>
-					</clip>
-					<noise>
-						<type>gaussian</type>
-						<mean>0.0</mean>
-						<stddev>0.007</stddev>
-					</noise>
-				</camera>
-				<plugin name="stereo_camera_controller" filename="libgazebo_ros_multicamera.so">
-					<alwaysOn>true</alwaysOn>
-					<cameraName>${prefix}</cameraName>
-					<imageTopicName>image_raw</imageTopicName>
-					<cameraInfoTopicName>camera_info</cameraInfoTopicName>
-					<frameName>${prefix}_base_link</frameName>
-					<hackBaseline>${baseline}</hackBaseline>
-					<distortionK1>0.0</distortionK1>
-					<distortionK2>0.0</distortionK2>
-					<distortionK3>0.0</distortionK3>
-					<distortionT1>0.0</distortionT1>
-					<distortionT2>0.0</distortionT2>
-					<ignoreTfPrefix>1</ignoreTfPrefix>
-				</plugin>
-			</sensor>
-		</gazebo>
-	</xacro:macro>
-	-->
-	<!--
-	<xacro:stereo_camera
-		prefix="${prefix}"
-		hfov="1.2217"
-		baseline="${baseline}"
-		fps="40"
-		width="640"
-		height="480"
-		format="${format}"
-		near="${near}"
-		far="${far}" />
-	-->
 </robot>

File: xacro/zed_mini.gazebo.xacro (robot description, xacro)
@@ -1,4 +1,3 @@
 <?xml version="1.0"?>
-<!-- Copyright (C) 2024, Federico Rollo -->
 <robot xmlns:xacro="http://ros.org/wiki/xacro">
   <xacro:macro name="gazebo_zedm" params="camera_name reference_frame baseline left_depth_optical_frame
@@ -6,7 +5,5 @@
   gyro_frame camera_center odom_frame odom_frame_joint robot_name
   disable_lumping:=true" >
-    <!-- Load parameters to model's main link-->
     <xacro:property name="deg_to_rad" value="0.01745329251994329577" />
-    <!-- LEFT CAMERA WITH DEPTH -->
     <gazebo reference="${left_color_optical_frame}">
       <sensor name="left_camera" type="depth">
@@ -39,5 +36,4 @@
           <pointCloudCutoff>0.3</pointCloudCutoff>
           <pointCloudCutoffMax>15.0</pointCloudCutoffMax>
-          <!-- TODO modify intrinsic params -->
           <distortionK1>0.00000001</distortionK1>
           <distortionK2>0.00000001</distortionK2>
@@ -53,6 +49,5 @@
       </sensor>
     </gazebo>
-    <!-- RIGHT CAMERA -->
-        <gazebo reference="${right_color_optical_frame}">
+    <gazebo reference="${right_color_optical_frame}">
       <sensor name="right_camera" type="depth">
         <update_rate>30</update_rate>
@@ -84,5 +79,4 @@
           <pointCloudCutoff>0.3</pointCloudCutoff>
           <pointCloudCutoffMax>15.0</pointCloudCutoffMax>
-          <!-- TODO modify intrinsic params -->
           <distortionK1>0.00000001</distortionK1>
           <distortionK2>0.00000001</distortionK2>
@@ -98,5 +92,4 @@
       </sensor>
     </gazebo>
-    <!-- IMU -->
     <gazebo reference="${gyro_frame}">
         <gravity>true</gravity>
@@ -117,5 +110,4 @@
         </sensor>
     </gazebo>
-    <!-- ODOMETRY -->
     <gazebo reference="${odom_frame_joint}">
         <disableFixedJointLumping>${disable_lumping}</disableFixedJointLumping>
